File: kicad/current_version/working/working.kicad_sch (KiCad schematic)
At the start: 6 parts, among them J1 h4psmra, U1 insoic14wi2cheli, U1 isn280

Commit message: commiting after auto generation
Parts:
- removed U1: isn280, oomlout_oomp_part_footprints:isn280_electronic_ic_lga_2_5_mm_x_2_5_mm_8_pin_sensor_pressure_temperature_bosch_bme280, symbol oomlout_oomp_part_symbols:isn280_electronic_ic_lga_2_5_mm_x_2_5_mm_8_pin_sensor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
- added J2: isnpt280, oomlout_oomp_part_footprints:isnpt280_electronic_ic_lga_8_pin_2_5_mm_x_2_5_mm_sensor_pressure_temperature_bosch_bme280, symbol oomlout_oomp_part_symbols:isnpt280_electronic_ic_lga_8_pin_2_5_mm_x_2_5_mm_sens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
Connections:
- net +3V3: now also J2.2 (CSB), J2.6 (VDDIO), J2.8 (VDD)
- net GND: now also J2.1 (GND), J2.7 (GND)
- net address: now also J2.5 (SDO)
- net scl_3v3: now also J2.4 (SCK)
- net sda_3v3: now also J2.3 (SDI)
Changed lines of the file:
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@@
-    )
-  )
-  (symbol (lib_id "oomlout_oomp_part_symbols:isn280_electronic_ic_lga_2_5_mm_x_2_5_mm_8_pin_sensor_pressure_temperature_bosch_bme280") (at 110.49 66.04 0) (unit 1)
-    (in_bom yes) (on_board yes) (dnp no)
-    (property "Reference" "U1" (at 111.76 64.77 0)
-      (effects (font (size 1.27 1.27)) (justify right))
-    )
-    (property "Value" "isn280" (at 111.76 67.31 0)
-      (effects (font (size 1.27 1.27)) (justify right))
-    )
-    (property "Footprint" "oomlout_oomp_part_footprints:isn280_electronic_ic_lga_2_5_mm_x_2_5_mm_8_pin_sensor_pressure_temperature_bosch_bme280" (at 148.59 77.47 0)
-      (effects (font (size 1.27 1.27)) hide)
-    )
-    (property "Datasheet" "https://github.com/oomlout/oomlout_oomp_v3/parts/electronic_ic_lga_2_5_mm_x_2_5_mm_8_pin_sensor_pressure_temperature_bosch_bme280/datasheet.pdf" (at 110.49 71.12 0)
-      (effects (font (size 1.27 1.27)) hide)
-    )
-    (pin "1")
-    (pin "2")
-    (pin "3")
-    (pin "4")
-    (pin "5")
-    (pin "6")
-    (pin "7")
-    (pin "8")
-    (instances
-      (project "working"
-        (path "/c9993764-076f-44f6-bf4c-6b69ce17c9e4"
-          (reference "U1") (unit 1)
-        )
-      )
-      (project "working"
-        (path "/e38c2552-f82c-42fa-b469-99aeb5e65e37"
-          (reference "U1") (unit 1)
-        )
-      )
     )
   )
@@
         )
       )
+    )
+  )
+  (symbol (lib_id "oomlout_oomp_part_symbols:isnpt280_electronic_ic_lga_8_pin_2_5_mm_x_2_5_mm_sensor_pressure_temperature_bosch_bme280") (at 110.49 66.04 0) (unit 1)
+    (in_bom yes) (on_board yes) (dnp no) (fields_autoplaced)
+    (property "Reference" "J2" (at 99.06 64.77 0)
+      (effects (font (size 1.27 1.27)) (justify right))
+    )
+    (property "Value" "isnpt280" (at 99.06 67.31 0)
+      (effects (font (size 1.27 1.27)) (justify right))
+    )
+    (property "Footprint" "oomlout_oomp_part_footprints:isnpt280_electronic_ic_lga_8_pin_2_5_mm_x_2_5_mm_sensor_pressure_temperature_bosch_bme280" (at 148.59 77.47 0)
+      (effects (font (size 1.27 1.27)) hide)
+    )
+    (property "Datasheet" "https://github.com/oomlout/oomlout_oomp_v3/parts/electronic_ic_lga_8_pin_2_5_mm_x_2_5_mm_sensor_pressure_temperature_bosch_bme280/datasheet.pdf" (at 110.49 71.12 0)
+      (effects (font (size 1.27 1.27)) hide)
+    )
+    (pin "1")
+    (pin "2")
+    (pin "3")
+    (pin "4")
+    (pin "5")
+    (pin "6")
+    (pin "7")
+    (pin "8")
+    (instances
+      (project "working"
+        (path "/e38c2552-f82c-42fa-b469-99aeb5e65e37"
+          (reference "J2") (unit 1)
+        )
+      )

Commit message: commiting after auto generation
Parts:
- removed J1: h4psmra, oomlout_oomp_part_footprints:h4psmra_electronic_header_1_mm_jst_sh_4_pin_surface_mount_right_angle, symbol oomlout_oomp_part_symbols:h4psmra_electronic_header_1_mm_jst_sh_4_pin_surface_m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
- removed J2: isnpt280, oomlout_oomp_part_footprints:isnpt280_electronic_ic_lga_8_pin_2_5_mm_x_2_5_mm_sensor_pressure_temperature_bosch_bme280, symbol oomlout_oomp_part_symbols:isnpt280_electronic_ic_lga_8_pin_2_5_mm_x_2_5_mm_sens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
- added CONN1: h4psmra, oomlout_oomp_part_footprints:h4psmra_electronic_header_1_mm_jst_sh_4_pin_surface_mount_right_angle, symbol oomlout_oomp_part_symbols:h4psmra_electronic_header_1_mm_jst_sh_4_pin_surface_m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
- added U1: isnpt280, oomlout_oomp_part_footprints:isnpt280_electronic_ic_lga_8_pin_2_5_mm_x_2_5_mm_sensor_pressure_temperature_bosch_bme280, symbol oomlout_oomp_part_symbols:isnpt280_electronic_ic_lga_8_pin_2_5_mm_x_2_5_mm_sens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
Connections:
- net +3V3: now also CONN1.3 (Pin_3), U1.2 (CSB), U1.6 (VDDIO), U1.8 (VDD)
- net GND: now also CONN1.4 (Pin_4), U1.1 (GND), U1.7 (GND)
- net address: now also U1.5 (SDO)
- net scl_3v3: now also CONN1.1 (Pin_1), U1.4 (SCK)
- net sda_3v3: now also CONN1.2 (Pin_2), U1.3 (SDI)
Changed lines of the file:
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@@
-    )
-  )
-  (symbol (lib_id "oomlout_oomp_part_symbols:h4psmra_electronic_header_1_mm_jst_sh_4_pin_surface_mount_right_angle") (at 175.26 46.99 0) (mirror x) (unit 1)
-    (in_bom yes) (on_board yes) (dnp no)
-    (property "Reference" "J1" (at 165.1 46.99 0)
-      (effects (font (size 1.27 1.27)))
-    )
-    (property "Value" "h4psmra" (at 165.1 44.45 0)
-      (effects (font (size 1.27 1.27)))
-    )
-    (property "Footprint" "oomlout_oomp_part_footprints:h4psmra_electronic_header_1_mm_jst_sh_4_pin_surface_mount_right_angle" (at 175.26 46.99 0)
-      (effects (font (size 1.27 1.27)) hide)
-    )
-    (property "Datasheet" "https://github.com/oomlout/oomlout_oomp_v3/parts/electronic_header_1_mm_jst_sh_4_pin_surface_mount_right_angle/datasheet.pdf" (at 175.26 46.99 0)
-      (effects (font (size 1.27 1.27)) hide)
-    )
-    (pin "1")
-    (pin "2")
-    (pin "3")
-    (pin "4")
-    (instances
-      (project "working"
-        (path "/c9993764-076f-44f6-bf4c-6b69ce17c9e4"
-          (reference "J1") (unit 1)
-        )
-      )
-      (project "working"
-        (path "/e38c2552-f82c-42fa-b469-99aeb5e65e37"
-          (reference "J1") (unit 1)
-        )
-      )
-    )
-  )
-  (symbol (lib_id "oomlout_oomp_part_symbols:isnpt280_electronic_ic_lga_8_pin_2_5_mm_x_2_5_mm_sensor_pressure_temperature_bosch_bme280") (at 110.49 66.04 0) (unit 1)
-    (in_bom yes) (on_board yes) (dnp no) (fields_autoplaced)
-    (property "Reference" "J2" (at 99.06 64.77 0)
-      (effects (font (size 1.27 1.27)) (justify right))
-    )
-    (property "Value" "isnpt280" (at 99.06 67.31 0)
-      (effects (font (size 1.27 1.27)) (justify right))
-    )
-    (property "Footprint" "oomlout_oomp_part_footprints:isnpt280_electronic_ic_lga_8_pin_2_5_mm_x_2_5_mm_sensor_pressure_temperature_bosch_bme280" (at 148.59 77.47 0)
-      (effects (font (size 1.27 1.27)) hide)
-    )
-    (property "Datasheet" "https://github.com/oomlout/oomlout_oomp_v3/parts/electronic_ic_lga_8_pin_2_5_mm_x_2_5_mm_sensor_pressure_temperature_bosch_bme280/datasheet.pdf" (at 110.49 71.12 0)
-      (effects (font (size 1.27 1.27)) hide)
-    )
-    (pin "1")
-    (pin "2")
-    (pin "3")
-    (pin "4")
-    (pin "5")
-    (pin "6")
-    (pin "7")
-    (pin "8")
-    (instances
-      (project "working"
-        (path "/e38c2552-f82c-42fa-b469-99aeb5e65e37"
-          (reference "J2") (unit 1)
-        )
-      )
     )
   )
@@
     (in_bom yes) (on_board yes) (dnp no)
     (property "Reference" "C2" (at 104.14 77.47 90)
-      (effects (font (size 1.27 1.27)))
+      (effects (font (size 1.27 1.27)) hide)
     )
     (property "Value" "c6nf100" (at 104.14 80.01 90)
@@
     )
   )
+  (symbol (lib_id "oomlout_oomp_part_symbols:h4psmra_electronic_header_1_mm_jst_sh_4_pin_surface_mount_right_angle") (at 175.26 44.45 0) (unit 1)
+    (in_bom yes) (on_board yes) (dnp no) (fields_autoplaced)
+    (property "Reference" "CONN1" (at 175.895 36.83 0)
+      (effects (font (size 1.27 1.27)))
+    )
+    (property "Value" "h4psmra" (at 175.895 39.37 0)
+      (effects (font (size 1.27 1.27)))
+    )
+    (property "Footprint" "oomlout_oomp_part_footprints:h4psmra_electronic_header_1_mm_jst_sh_4_pin_surface_mount_right_angle" (at 175.26 44.45 0)
+      (effects (font (size 1.27 1.27)) hide)
+    )
+    (property "Datasheet" "https://github.com/oomlout/oomlout_oomp_v3/parts/electronic_header_1_mm_jst_sh_4_pin_surface_mount_right_angle/datasheet.pdf" (at 175.26 44.45 0)
+      (effects (font (size 1.27 1.27)) hide)
+    )
+    (pin "1")
+    (pin "2")
+    (pin "3")
+    (pin "4")
+    (instances
+      (project "working"
+        (path "/e38c2552-f82c-42fa-b469-99aeb5e65e37"
+          (reference "CONN1") (unit 1)
+        )
+      )
+    )
+  )
   (symbol (lib_id "power:+3V3") (at 193.04 39.37 0) (unit 1)
     (in_bom yes) (on_board yes) (dnp no) (fields_autoplaced)
@@
         )
       )
+    )
+  )
+  (symbol (lib_id "oomlout_oomp_part_symbols:isnpt280_electronic_ic_lga_8_pin_2_5_mm_x_2_5_mm_sensor_pressure_temperature_bosch_bme280") (at 110.49 66.04 0) (unit 1)
+    (in_bom yes) (on_board yes) (dnp no)
+    (property "Reference" "U1" (at 99.06 64.77 0)
+      (effects (font (size 1.27 1.27)) (justify right))
+    )
+    (property "Value" "isnpt280" (at 99.06 67.31 0)
+      (effects (font (size 1.27 1.27)) (justify right))
+    )
+    (property "Footprint" "oomlout_oomp_part_footprints:isnpt280_electronic_ic_lga_8_pin_2_5_mm_x_2_5_mm_sensor_pressure_temperature_bosch_bme280" (at 148.59 77.47 0)
+      (effects (font (size 1.27 1.27)) hide)
+    )
+    (property "Datasheet" "https://github.com/oomlout/oomlout_oomp_v3/parts/electronic_ic_lga_8_pin_2_5_mm_x_2_5_mm_sensor_pressure_temperature_bosch_bme280/datasheet.pdf" (at 110.49 71.12 0)
+      (effects (font (size 1.27 1.27)) hide)
+    )
+    (pin "1")
+    (pin "2")
+    (pin "3")
+    (pin "4")
+    (pin "5")
+    (pin "6")
+    (pin "7")
+    (pin "8")
+    (instances
+      (project "working"
+        (path "/e38c2552-f82c-42fa-b469-99aeb5e65e37"
+          (reference "U1") (unit 1)
+        )
+      )
